Commit message: remove unneeded plugins

File: pr2_description/gazebo/gazebo.urdf.xacro (robot description, xacro)
@@ -2,20 +2,20 @@
 <robot xmlns:xacro="http://ros.org/wiki/xacro">
   <gazebo>
-    <plugin name="gazebo_ros_controller_manager" filename="libgazebo_ros_controller_manager.so">
-      <alwaysOn>true</alwaysOn>
-      <updateRate>1000.0</updateRate>
-    </plugin>
-    <plugin name="gazebo_ros_power_monitor_controller" filename="libgazebo_ros_power_monitor.so">
-      <alwaysOn>true</alwaysOn>
-      <updateRate>1.0</updateRate>
-      <timeout>5</timeout>
-      <powerStateTopic>power_state</powerStateTopic>
-      <powerStateRate>10.0</powerStateRate>
-      <fullChargeCapacity>87.78</fullChargeCapacity>
-      <dischargeRate>-474</dischargeRate>
-      <chargeRate>525</chargeRate>
-      <dischargeVoltage>15.52</dischargeVoltage>
-      <chargeVoltage>16.41</chargeVoltage>
-    </plugin>
+    <!-- <plugin name="gazebo_ros_controller_manager" filename="libgazebo_ros_controller_manager.so"> -->
+    <!--   <alwaysOn>true</alwaysOn> -->
+    <!--   <updateRate>1000.0</updateRate> -->
+    <!-- </plugin> -->
+    <!-- <plugin name="gazebo_ros_power_monitor_controller" filename="libgazebo_ros_power_monitor.so"> -->
+    <!--   <alwaysOn>true</alwaysOn> -->
+    <!--   <updateRate>1.0</updateRate> -->
+    <!--   <timeout>5</timeout> -->
+    <!--   <powerStateTopic>power_state</powerStateTopic> -->
+    <!--   <powerStateRate>10.0</powerStateRate> -->
+    <!--   <fullChargeCapacity>87.78</fullChargeCapacity>      -->
+    <!--   <dischargeRate>-474</dischargeRate> -->
+    <!--   <chargeRate>525</chargeRate> -->
+    <!--   <dischargeVoltage>15.52</dischargeVoltage> -->
+    <!--   <chargeVoltage>16.41</chargeVoltage> -->
+    <!-- </plugin> -->
     <plugin name="gazebo_force_set_joint_position" filename="libgazebo_force_set_joint_position.so"/>
   </gazebo>

File: pr2_description/urdf/sensors/projector_wg6802418.gazebo.xacro (robot description, xacro)
@@ -4,25 +4,25 @@
      this will only work with added r36415 patch in simulator_gazebo stack
      otherwise projector will not work without removing the reference tag -->
-<xacro:macro name="projector_wg6802418_gazebo_v0" params="name">
-  <gazebo reference="${name}_child_frame">
-    <projector name="${name}_projector_wg6802418">
-      <pose>0 0 0 0 -1.5707 0</pose>
-      <texture>stereo_projection_pattern_high_res_red.png</texture>
-      <fov>${55.0/180.0*M_PI}</fov>
-      <near_clip>0.1</near_clip>
-      <far_clip>10</far_clip>
-    </projector>
-  </gazebo>
-  <gazebo>
-    <plugin name="${name}_controller" filename="libgazebo_ros_projector.so">
-      <projector>${name}_child_frame/${name}_projector_wg6802418</projector>
-      <alwaysOn>true</alwaysOn>
-      <updateRate>15.0</updateRate>
-      <textureName>stereo_projection_pattern_high_res_red.png</textureName>
-      <filterTextureName>stereo_projection_pattern_filter.png</filterTextureName>
-      <textureTopicName>${name}_controller/image</textureTopicName>
-      <projectorTopicName>${name}_controller/projector</projectorTopicName>
-    </plugin>
-  </gazebo>
-</xacro:macro>
+<!-- <xacro:macro name="projector_wg6802418_gazebo_v0" params="name"> -->
+  <!-- <gazebo reference="${name}_child_frame"> -->
+  <!--   <projector name="${name}_projector_wg6802418"> -->
+  <!--     <pose>0 0 0 0 -1.5707 0</pose> -->
+  <!--     <texture>stereo_projection_pattern_high_res_red.png</texture> -->
+  <!--     <fov>${55.0/180.0*M_PI}</fov> -->
+  <!--     <near_clip>0.1</near_clip> -->
+  <!--     <far_clip>10</far_clip> -->
+  <!--   </projector> -->
+  <!-- </gazebo> -->
+  <!-- <gazebo> -->
+    <!-- <plugin name="${name}_controller" filename="libgazebo_ros_projector.so"> -->
+    <!--   <projector>${name}_child_frame/${name}_projector_wg6802418</projector> -->
+    <!--   <alwaysOn>true</alwaysOn> -->
+    <!--   <updateRate>15.0</updateRate> -->
+    <!--   <textureName>stereo_projection_pattern_high_res_red.png</textureName> -->
+    <!--   <filterTextureName>stereo_projection_pattern_filter.png</filterTextureName>         -->
+    <!--   <textureTopicName>${name}_controller/image</textureTopicName> -->
+    <!--   <projectorTopicName>${name}_controller/projector</projectorTopicName> -->
+    <!-- </plugin> -->
+  <!-- </gazebo> -->
+<!-- </xacro:macro> -->
 </root>

File: pr2_description/urdf/sensors/prosilica_gc2450_camera.gazebo.xacro (robot description, xacro)
@@ -1,41 +1,41 @@
 <?xml version="1.0"?>
 <root xmlns:xacro="http://ros.org/wiki/xacro">
-<xacro:macro name="prosilica_cam_gazebo_v0" params="camera_name frame_name">
-  <gazebo reference="${frame_name}_frame">
-    <sensor type="camera" name="${frame_name}_sensor">
-      <always_on>true</always_on>
-      <update_rate>20.0</update_rate>
-      <camera>
-        <horizontal_fov>${M_PI/4}</horizontal_fov>
-        <image>
-          <format>R8G8B8</format>
-          <width>2448</width>
-          <height>2050</height>
-        </image>
-        <clip>
-          <near>0.1</near>
-          <far>100</far>
-        </clip>
-      </camera>
-      <plugin name="${frame_name}_controller" filename="libgazebo_ros_prosilica.so">
-        <updateRate>20.0</updateRate>
-        <cameraName>${camera_name}</cameraName>
-        <imageTopicName>image_raw</imageTopicName>
-        <cameraInfoTopicName>camera_info</cameraInfoTopicName>
-        <pollServiceName>request_image</pollServiceName>
-        <frameName>${frame_name}_optical_frame</frameName>
-        <CxPrime>1224.5</CxPrime>
-        <Cx>1224.5</Cx>
-        <Cy>1025.5</Cy>
-        <focalLength>2954.998083</focalLength>
-        <distortionK1>0.0</distortionK1>
-        <distortionK2>0.0</distortionK2>
-        <distortionK3>0.0</distortionK3>
-        <distortionT1>0.0</distortionT1>
-        <distortionT2>0.0</distortionT2>
-      </plugin>
-    </sensor>
-    <material value="Gazebo/Black" />
-  </gazebo>
-</xacro:macro>
+<!-- <xacro:macro name="prosilica_cam_gazebo_v0" params="camera_name frame_name"> -->
+<!--   <gazebo reference="${frame_name}_frame"> -->
+<!--     <sensor type="camera" name="${frame_name}_sensor"> -->
+<!--       <always_on>true</always_on> -->
+<!--       <update_rate>20.0</update_rate> -->
+<!--       <camera> -->
+<!--         <horizontal_fov>${M_PI/4}</horizontal_fov> -->
+<!--         <image> -->
+<!--           <format>R8G8B8</format> -->
+<!--           <width>2448</width> -->
+<!--           <height>2050</height> -->
+<!--         </image> -->
+<!--         <clip> -->
+<!--           <near>0.1</near> -->
+<!--           <far>100</far> -->
+<!--         </clip> -->
+<!--       </camera> -->
+<!--       <plugin name="${frame_name}_controller" filename="libgazebo_ros_prosilica.so"> -->
+<!--         <updateRate>20.0</updateRate> -->
+<!--         <cameraName>${camera_name}</cameraName> -->
+<!--         <imageTopicName>image_raw</imageTopicName> -->
+<!--         <cameraInfoTopicName>camera_info</cameraInfoTopicName> -->
+<!--         <pollServiceName>request_image</pollServiceName> -->
+<!--         <frameName>${frame_name}_optical_frame</frameName> -->
+<!--         <CxPrime>1224.5</CxPrime> -->
+<!--         <Cx>1224.5</Cx> -->
+<!--         <Cy>1025.5</Cy> -->
+<!--         <focalLength>2954.998083</focalLength> -->
+<!--         <distortionK1>0.0</distortionK1> -->
+<!--         <distortionK2>0.0</distortionK2> -->
+<!--         <distortionK3>0.0</distortionK3> -->
+<!--         <distortionT1>0.0</distortionT1> -->
+<!--         <distortionT2>0.0</distortionT2> -->
+<!--       </plugin> -->
+<!--     </sensor> -->
+<!--     <material value="Gazebo/Black" /> -->
+<!--   </gazebo> -->
+<!-- </xacro:macro> -->
 </root>

File: pr2_description/urdf/sensors/wge100_camera.gazebo.xacro (robot description, xacro)
@@ -1,45 +1,43 @@
 <?xml version="1.0"?>
 <robot xmlns:xacro="http://ros.org/wiki/xacro">
-  <xacro:macro name="wge100_camera_gazebo_v0" params="name camera_name image_format image_topic_name camera_info_topic_name hfov focal_length frame_id hack_baseline image_width image_height">
-    <gazebo reference="${name}_frame">
-      <sensor type="camera" name="${name}_sensor">
-        <always_on>true</always_on>
-        <update_rate>25.0</update_rate>
-        <camera>
-          <horizontal_fov>${hfov*M_PI/180.0}</horizontal_fov>
-          <image>
-            <format>${image_format}</format>
-            <width>${image_width}</width>
-            <height>${image_height}</height>
-          </image>
-          <clip>
-            <near>0.1</near>
-            <far>100</far>
-          </clip>
-        </camera>
-        <plugin name="${name}_controller" filename="libgazebo_ros_camera.so">
-          <alwaysOn>true</alwaysOn>
-          <updateRate>25.0</updateRate>
-          <cameraName>${camera_name}</cameraName>
-          <imageTopicName>${image_topic_name}</imageTopicName>
-          <cameraInfoTopicName>${camera_info_topic_name}</cameraInfoTopicName>
-          <frameName>${frame_id}</frameName>
-          <hackBaseline>${hack_baseline}</hackBaseline>
-          <CxPrime>${(image_width+1)/2}</CxPrime>
-          <Cx>${(image_width+1)/2}</Cx>
-          <Cy>${(image_height+1)/2}</Cy>
-          <!-- image_width / (2*tan(hfov_radian /2)) -->
-          <!-- 320 for wide and 772.55 for narrow stereo camera -->
-          <focalLength>${focal_length}</focalLength>
-          <distortionK1>0.0</distortionK1>
-          <distortionK2>0.0</distortionK2>
-          <distortionK3>0.0</distortionK3>
-          <distortionT1>0.0</distortionT1>
-          <distortionT2>0.0</distortionT2>
-        </plugin>
-      </sensor>
-      <turnGravityOff>true</turnGravityOff>
-      <material>PR2/Blue</material>
-    </gazebo>
-  </xacro:macro>
+  <!-- <xacro:macro name="wge100_camera_gazebo_v0" params="name camera_name image_format image_topic_name camera_info_topic_name hfov focal_length frame_id hack_baseline image_width image_height"> -->
+  <!--   <gazebo reference="${name}_frame"> -->
+  <!--     <sensor type="camera" name="${name}_sensor"> -->
+  <!--       <always_on>true</always_on> -->
+  <!--       <update_rate>25.0</update_rate> -->
+  <!--       <camera> -->
+  <!--         <horizontal_fov>${hfov*M_PI/180.0}</horizontal_fov> -->
+  <!--         <image> -->
+  <!--           <format>${image_format}</format> -->
+  <!--           <width>${image_width}</width> -->
+  <!--           <height>${image_height}</height> -->
+  <!--         </image> -->
+  <!--         <clip> -->
+  <!--           <near>0.1</near> -->
+  <!--           <far>100</far> -->
+  <!--         </clip> -->
+  <!--       </camera> -->
+  <!--       <plugin name="${name}_controller" filename="libgazebo_ros_camera.so"> -->
+  <!--         <alwaysOn>true</alwaysOn> -->
+  <!--         <updateRate>25.0</updateRate> -->
+  <!--         <cameraName>${camera_name}</cameraName> -->
+  <!--         <imageTopicName>${image_topic_name}</imageTopicName> -->
+  <!--         <cameraInfoTopicName>${camera_info_topic_name}</cameraInfoTopicName> -->
+  <!--         <frameName>${frame_id}</frameName> -->
+  <!--         <hackBaseline>${hack_baseline}</hackBaseline> -->
+  <!--         <CxPrime>${(image_width+1)/2}</CxPrime> -->
+  <!--         <Cx>${(image_width+1)/2}</Cx> -->
+  <!--         <Cy>${(image_height+1)/2}</Cy> -->
+  <!--         <focalLength>${focal_length}</focalLength> -->
+  <!--         <distortionK1>0.0</distortionK1> -->
+  <!--         <distortionK2>0.0</distortionK2> -->
+  <!--         <distortionK3>0.0</distortionK3> -->
+  <!--         <distortionT1>0.0</distortionT1> -->
+  <!--         <distortionT2>0.0</distortionT2> -->
+  <!--       </plugin> -->
+  <!--     </sensor> -->
+  <!--     <turnGravityOff>true</turnGravityOff> -->
+  <!--     <material>PR2/Blue</material> -->
+  <!--   </gazebo> -->
+  <!-- </xacro:macro> -->
 </robot>
