Commit message: update

File: pr2_description/urdf/gripper_v0/gripper.gazebo.xacro (robot description, xacro)
@@ -48,16 +48,4 @@
       <turnGravityOff>true</turnGravityOff>
       <selfCollide>false</selfCollide>
-      <sensor type="contact" name="${prefix}_l_finger_tip_contact_sensor">
-        <update_rate>100.0</update_rate>
-        <contact>
-          <collision>${prefix}_l_finger_tip_link_collision</collision>
-        </contact>
-        <plugin name="${prefix}_l_finger_tip_gazebo_ros_bumper_controller" filename="libgazebo_ros_bumper.so">
-          <alwaysOn>true</alwaysOn>
-          <frameName>${prefix}_l_finger_tip_link</frameName>
-          <updateRate>100.0</updateRate>
-          <bumperTopicName>${prefix}_l_finger_tip_bumper</bumperTopicName>
-        </plugin>
-      </sensor>
       <mu1 value="${finger_tip_mu}" />
       <mu2 value="${finger_tip_mu}" />
@@ -75,16 +63,4 @@
       <turnGravityOff>true</turnGravityOff>
       <selfCollide>false</selfCollide>
-      <sensor type="contact" name="${prefix}_r_finger_tip_contact_sensor">
-        <update_rate>100.0</update_rate>
-        <contact>
-          <collision>${prefix}_r_finger_tip_link_collision</collision>
-        </contact>
-        <plugin name="${prefix}_r_finger_tip_gazebo_ros_bumper_controller" filename="libgazebo_ros_bumper.so">
-          <alwaysOn>true</alwaysOn>
-          <frameName>${prefix}_r_finger_tip_link</frameName>
-          <updateRate>100.0</updateRate>
-          <bumperTopicName>${prefix}_r_finger_tip_bumper</bumperTopicName>
-        </plugin>
-      </sensor>
       <mu1 value="${finger_tip_mu}" />
       <mu2 value="${finger_tip_mu}" />
@@ -93,18 +69,4 @@
     </gazebo>
     <gazebo>
-      <plugin name="p3d_${prefix}_l_finger_controller" filename="libgazebo_ros_p3d.so">
-        <alwaysOn>true</alwaysOn>
-        <updateRate>100.0</updateRate>
-        <bodyName>${prefix}_l_finger_link</bodyName>
-        <topicName>${prefix}_l_finger_pose_ground_truth</topicName>
-        <gaussianNoise>0.0</gaussianNoise>
-        <frameName>base_link</frameName>
-      </plugin>
-      <plugin name="f3d_${prefix}_l_finger_controller" filename="libgazebo_ros_f3d.so">
-        <alwaysOn>true</alwaysOn>
-        <updateRate>100.0</updateRate>
-        <bodyName>${prefix}_l_finger_link</bodyName>
-        <topicName>${prefix}_l_finger_force_ground_truth</topicName>
-      </plugin>
     </gazebo>
     <gazebo reference="${prefix}_r_finger_tip_joint">
@@ -236,14 +198,4 @@
     </gazebo>
     <gazebo>
-      <plugin name="p3d_${side}_gripper_palm_controller" filename="libgazebo_ros_p3d.so">
-        <alwaysOn>true</alwaysOn>
-        <updateRate>100.0</updateRate>
-        <bodyName>${side}_gripper_palm_link</bodyName>
-        <topicName>${side}_gripper_palm_pose_ground_truth</topicName>
-        <xyzOffsets>0 0 0</xyzOffsets>
-        <rpyOffsets>0 0 0</rpyOffsets>
-        <gaussianNoise>0.0</gaussianNoise>
-        <frameName>map</frameName>
-      </plugin>
       <!-- a formal implementation of grasp hack in gazebo with fixed joint -->
       <gripper name="${side}_grasp_hack">

File: pr2_description/urdf/sensors/kinect_prosilica_camera.gazebo.xacro (robot description, xacro)
@@ -103,85 +103,3 @@
   </transmission>
 </xacro:macro>
-<xacro:macro name="prosilica_cam_gazebo_v1" params="link_name frame_name camera_name ">
-  <gazebo reference="${link_name}">
-    <sensor type="camera" name="${link_name}_sensor">
-      <always_on>true</always_on>
-      <update_rate>1.0</update_rate>
-      <camera>
-        <horizontal_fov>${64.2*M_PI/180.0}</horizontal_fov>
-        <image>
-          <format>R8G8B8</format>
-          <width>320</width>
-          <height>240</height>
-        </image>
-        <clip>
-          <near>0.1</near>
-          <far>100</far>
-        </clip>
-      </camera>
-      <plugin name="${link_name}_controller" filename="libgazebo_ros_prosilica.so">
-        <alwaysOn>true</alwaysOn>
-        <updateRate>1.0</updateRate>
-        <cameraName>${camera_name}_1mb</cameraName>
-        <imageTopicName>image_raw</imageTopicName>
-        <cameraInfoTopicName>camera_info</cameraInfoTopicName>
-        <depthImageTopicName>depth/image_raw</depthImageTopicName>
-        <depthImageCameraInfoTopicName>depth/camera_info</depthImageCameraInfoTopicName>
-        <pollServiceName>request_image</pollServiceName>
-        <pointCloudTopicName>points</pointCloudTopicName>
-        <frameName>${frame_name}</frameName>
-        <pointCloudCutoff>0.4</pointCloudCutoff>
-        <distortionK1>0.0</distortionK1>
-        <distortionK2>0.0</distortionK2>
-        <distortionK3>0.0</distortionK3>
-        <distortionT1>0.0</distortionT1>
-        <distortionT2>0.0</distortionT2>
-        <CxPrime>0</CxPrime>
-        <Cx>0</Cx>
-        <Cy>0</Cy>
-        <focalLength>0</focalLength>
-        <hackBaseline>0</hackBaseline>
-      </plugin>
-    </sensor>
-    <sensor type="depth" name="${link_name}_sim_pcd_sensor">
-      <always_on>true</always_on>
-      <update_rate>1.0</update_rate>
-      <camera>
-        <horizontal_fov>${64.2*M_PI/180.0}</horizontal_fov>
-        <image>
-          <format>R8G8B8</format>
-          <width>320</width>
-          <height>240</height>
-        </image>
-        <clip>
-          <near>0.1</near>
-          <far>100</far>
-        </clip>
-      </camera>
-      <plugin name="${link_name}_sim_pcd_controller" filename="libgazebo_ros_openni_kinect.so">
-        <alwaysOn>true</alwaysOn>
-        <updateRate>1.0</updateRate>
-        <cameraName>${camera_name}_1mb_sim_pcd</cameraName>
-        <imageTopicName>image_raw</imageTopicName>
-        <depthImageTopicName>depth/image_raw</depthImageTopicName>
-        <depthImageCameraInfoTopicName>depth/camera_info</depthImageCameraInfoTopicName>
-        <cameraInfoTopicName>camera_info</cameraInfoTopicName>
-        <pointCloudTopicName>points</pointCloudTopicName>
-        <frameName>${frame_name}</frameName>
-        <pointCloudCutoff>0.4</pointCloudCutoff>
-        <distortionK1>0.00000001</distortionK1>
-        <distortionK2>0.00000001</distortionK2>
-        <distortionK3>0.00000001</distortionK3>
-        <distortionT1>0.00000001</distortionT1>
-        <distortionT2>0.00000001</distortionT2>
-        <CxPrime>0</CxPrime>
-        <Cx>0</Cx>
-        <Cy>0</Cy>
-        <focalLength>0</focalLength>
-        <hackBaseline>0</hackBaseline>
-      </plugin>
-    </sensor>
-    <material value="Gazebo/Red" />
-  </gazebo>
-</xacro:macro>
 </root>
